File: Drone_PCB/Drone_PCB.sch (KiCad schematic (older format))
At the start: 38 parts, among them J1 Conn_01x02, J2 Conn_01x02, J3 Conn_01x02, J4 Conn_01x02, J5 USB_B_Mini, Q1 TRANS_NPN-MMBT2222AL, Q2 TRANS_NPN-MMBT2222AL, U1 ESP32-WROOM-32, U2 CP2104, U3 L293D, U4 MIC5219-3.3YMM, U5 L293D, U6 MPU-6050, U7 MCP73832-2-OT

Commit message: V2 - With Mosfets
Removed the H-Bridge added the MOSFETS
Parts:
- removed C4: 10uF, symbol Device:C_Small
- removed C5: 0.1uF, symbol Device:C_Small
- removed C6: 4.7uF, symbol Device:C_Small
- removed D1: LED, symbol Device:LED
- removed R1: 2K2, symbol Device:R_Small
- removed R2: 470R, symbol Device:R_Small
- removed U3, U5: L293D, Package_DIP:DIP-16_W7.62mm, symbol Driver_Motor:L293D
- removed U7: MCP73832-2-OT, Package_TO_SOT_SMD:SOT-23-5, symbol Battery_Management:MCP73832-2-OT
- added D2, D3, D4, D5: D_Schottky, symbol Device:D_Schottky
- added J6, J7, J8: Conn_01x05, Connector_PinHeader_2.54mm:PinHeader_1x05_P2.54mm_Vertical, symbol Connector_Generic:Conn_01x05
- added R10, R11: 2k2, Resistor_SMD:R_0603_1608Metric_Pad1.05x0.95mm_HandSolder, symbol Device:R_Small
- added R12, R13, R14, R15: 10K, Resistor_SMD:R_0603_1608Metric_Pad1.05x0.95mm_HandSolder, symbol Device:R_Small
- added R16, R17: 0R, Resistor_SMD:R_0603_1608Metric_Pad1.05x0.95mm_HandSolder, symbol Device:R_Small
- added U3, U5, U8, U9: SI2302-TP, Package_TO_SOT_SMD:SOT-23, symbol Drone_Lib:SI2302-TP
- C1, C10, C11, C12, C13, C2, C3, C7, C8, C9: footprint (none) -> Capacitor_SMD:C_0603_1608Metric_Pad1.05x0.95mm_HandSolder
- J5: footprint (none) -> Connector_USB:USB_Micro-B_Molex-105017-0001
- R3, R4, R5, R6, R7, R8, R9: footprint (none) -> Resistor_SMD:R_0603_1608Metric_Pad1.05x0.95mm_HandSolder
Connections:
- net labels added: AUX_SCL, AUX_SDA, IO25, IO26, IO27, IO32, IO33, M1_PWM, M2_PWM, M3_PWM, M4_PWM, SCK, SCS, SDI, SDO
- net labels removed: M1_IN1, M1_IN2, M2_IN1, M2_IN2, M3_IN1, M3_IN2, M4_IN1, M4_IN2
- wire segments 202 -> 236
Other:
- note added: "DO NOT POPULATE"
- note added: "Extra Development Signals"
- note added: "MOSFETS motor Drivers"
- note removed: "Battery Charger"
- note removed: "H-Bridge circuit"

Commit message: Routing Part 6
We made the tracks thicker and removed some components
Parts:
- removed J6, J7, J8: Conn_01x05, Connector_PinHeader_2.54mm:PinHeader_1x05_P2.54mm_Vertical, symbol Connector_Generic:Conn_01x05
- J5: footprint Connector_USB:USB_Micro-B_Molex-105017-0001 -> Connector_USB:USB_Micro-B_Molex_47346-0001
Connections:
- wire segments 236 -> 216
Other:
- note removed: "Extra Development Signals"
Changed lines of the file:
@@
 F 0 "J5" H 6557 3817 50  0000 C CNN
 F 1 "USB_B_Mini" H 6557 3726 50  0000 C CNN
-F 2 "Connector_USB:USB_Micro-B_Molex-105017-0001" H 6650 3300 50  0001 C CNN
+F 2 "Connector_USB:USB_Micro-B_Molex_47346-0001" H 6650 3300 50  0001 C CNN
 F 3 "https://www.molex.com/molex/products/part-detail/io_connectors/1050170001" H 6650 3300 50  0001 C CNN
 	1    6500 3350
@@
 	9550 5150 10000 5150
 Wire Wire Line
-	10200 4850 10650 4850
-Wire Wire Line
 	9350 5150 8900 5150
 Wire Wire Line
@@
 Text Label 8950 5950 0    50   ~ 0
 DTR
-Text Label 10450 6300 0    50   ~ 0
+Text Label 10700 6300 2    50   ~ 0
 RESET
-Text Label 10450 5450 0    50   ~ 0
+Text Label 10700 5450 2    50   ~ 0
 DTR
-Text Label 10400 4850 0    50   ~ 0
-GPIO0
 Text Label 9750 3200 0    50   ~ 0
 TX_CP2104
@@
 P 10400 3200
 F 0 "R5" V 10500 3250 50  0000 L CNN
-F 1 "100R" V 10500 3050 50  0000 L CNN
+F 1 "100R" V 10500 3000 50  0000 L CNN
 F 2 "Resistor_SMD:R_0603_1608Metric_Pad1.05x0.95mm_HandSolder" H 10400 3200 50  0001 C CNN
 F 3 "~" H 10400 3200 50  0001 C CNN
@@
 Wire Wire Line
 	10500 3300 10900 3300
-Wire Wire Line
-	10500 3200 10900 3200
-Text Label 10550 3200 0    50   ~ 0
-RX_ESP32
-Text Label 10550 3300 0    50   ~ 0
+Text Label 10900 3300 2    50   ~ 0
 TX_ESP32
 Wire Wire Line
@@
 Wire Wire Line
 	3600 3100 4000 3100
-Text Label 3650 3100 0    50   ~ 0
+Text Label 4000 3100 2    50   ~ 0
 RX_ESP32
-Text Label 3650 2900 0    50   ~ 0
+Text Label 4000 2900 2    50   ~ 0
 TX_ESP32
 $Comp
@@
 Wire Wire Line
 	9650 2900 10100 2900
-Text Label 9950 2900 0    50   ~ 0
+Text Label 10100 2900 2    50   ~ 0
 DTR
-Text Label 9950 3500 0    50   ~ 0
+Text Label 10100 3500 2    50   ~ 0
 RTS
 $Comp
@@
 	1850 3500 1850 3400
 Connection ~ 1750 3500
-$Comp
-L power:GND #PWR022
-U 1 1 5F349ABA
-P 3000 5650
-F 0 "#PWR022" H 3000 5400 50  0001 C CNN
-F 1 "GND" H 3005 5477 50  0000 C CNN
-F 2 "" H 3000 5650 50  0001 C CNN
-F 3 "" H 3000 5650 50  0001 C CNN
-	1    3000 5650
-	1    0    0    -1
-$EndComp
 Wire Wire Line
 	3000 5650 3000 5400
@@
 	1400 9100 1850 9100
 Wire Wire Line
-	1400 9200 1850 9200
-Wire Wire Line
 	1400 9350 1850 9350
 Wire Wire Line
@@
 Wire Wire Line
 	1400 9700 1850 9700
-Text Label 1700 8850 0    50   ~ 0
+Text Label 1850 8850 2    50   ~ 0
 M1+
-Text Label 1700 8950 0    50   ~ 0
+Text Label 1850 8950 2    50   ~ 0
 M1-
-Text Label 1700 9100 0    50   ~ 0
+Text Label 1850 9100 2    50   ~ 0
 M2+
-Text Label 1700 9200 0    50   ~ 0
-M2-
-Text Label 1700 9350 0    50   ~ 0
+Text Label 1850 9350 2    50   ~ 0
 M3+
-Text Label 1700 9450 0    50   ~ 0
+Text Label 1850 9450 2    50   ~ 0
 M3-
-Text Label 1700 9700 0    50   ~ 0
+Text Label 1850 9700 2    50   ~ 0
 M4-
-Text Label 1700 9600 0    50   ~ 0
+Text Label 1850 9600 2    50   ~ 0
 M4+
 Wire Notes Line
@@
 Wire Wire Line
 	4200 3600 3600 3600
-Wire Wire Line
-	4200 3500 3600 3500
 Text Label 4200 3600 2    50   ~ 0
 M1_PWM
@@
 Wire Wire Line
 	4200 3400 3600 3400
-Wire Wire Line
-	4200 3700 3600 3700
 Text Label 4200 3800 2    50   ~ 0
 M2_PWM
 Wire Wire Line
 	4200 3800 3600 3800
-Wire Wire Line
-	4200 3900 3600 3900
 Text Label 4200 3400 2    50   ~ 0
 M3_PWM
 Wire Wire Line
 	4200 4000 3600 4000
-Wire Wire Line
-	4200 4100 3600 4100
 Text Label 4200 4000 2    50   ~ 0
 M4_PWM
@@
 Wire Notes Line
 	5100 11000 11550 11000
-$Comp
-L Connector_Generic:Conn_01x05 J6
-U 1 1 5F977D5C
-P 14250 1700
-F 0 "J6" H 14330 1742 50  0000 L CNN
-F 1 "Conn_01x05" H 14330 1651 50  0000 L CNN
-F 2 "Connector_PinHeader_2.54mm:PinHeader_1x05_P2.54mm_Vertical" H 14250 1700 50  0001 C CNN
-F 3 "~" H 14250 1700 50  0001 C CNN
-	1    14250 1700
-	1    0    0    -1
-$EndComp
-Text Label 13750 1700 0    50   ~ 0
-SDA
-Text Label 13750 1600 0    50   ~ 0
-SCL
-Wire Wire Line
-	14050 1600 13750 1600
-Wire Wire Line
-	14050 1700 13750 1700
-$Comp
-L power:+3V3 #PWR05
-U 1 1 5F98648C
-P 13750 1300
-F 0 "#PWR05" H 13750 1150 50  0001 C CNN
-F 1 "+3V3" H 13765 1473 50  0000 C CNN
-F 2 "" H 13750 1300 50  0001 C CNN
-F 3 "" H 13750 1300 50  0001 C CNN
-	1    13750 1300
-	1    0    0    -1
-$EndComp
-Wire Wire Line
-	14050 1500 13750 1500
-Wire Wire Line
-	13750 1500 13750 1300
-$Comp
-L power:GND #PWR06
-U 1 1 5F9B9DF5
-P 13750 2000
-F 0 "#PWR06" H 13750 1750 50  0001 C CNN
-F 1 "GND" H 13755 1827 50  0000 C CNN
-F 2 "" H 13750 2000 50  0001 C CNN
-F 3 "" H 13750 2000 50  0001 C CNN
-	1    13750 2000
-	1    0    0    -1
-$EndComp
-Wire Wire Line
-	13750 2000 13750 1900
-Wire Wire Line
-	14050 1900 13750 1900
 Wire Wire Line
 	3600 4500 4000 4500
@@
 Text Label 15150 8200 2    49   ~ 0
 AUX_SCL
-Text Label 13500 1800 0    50   ~ 0
-V_BAT_Measure
-Wire Wire Line
-	14050 1800 13500 1800
-Wire Notes Line
-	15850 3600 12100 3600
-Wire Notes Line
-	12100 3600 12100 650
-Wire Notes Line
-	12100 650  15850 650
-Wire Notes Line
-	15850 650  15850 3600
-Text Notes 12800 900  0    118  ~ 0
-Extra Development Signals
-Wire Wire Line
-	14050 3250 13700 3250
-Wire Wire Line
-	14050 3150 13700 3150
-Text Label 13700 3150 0    49   ~ 0
-AUX_SCL
-Text Label 13700 3250 0    49   ~ 0
-AUX_SDA
-$Comp
-L Connector_Generic:Conn_01x05 J8
-U 1 1 5FBF3683
-P 14250 3050
-F 0 "J8" H 14330 3092 50  0000 L CNN
-F 1 "Conn_01x05" H 14330 3001 50  0000 L CNN
-F 2 "Connector_PinHeader_2.54mm:PinHeader_1x05_P2.54mm_Vertical" H 14250 3050 50  0001 C CNN
-F 3 "~" H 14250 3050 50  0001 C CNN
-	1    14250 3050
-	1    0    0    -1
-$EndComp
-Text Label 13700 3050 0    49   ~ 0
-SCK
-Text Label 13700 2950 0    49   ~ 0
-SDI
-Text Label 13700 2850 0    49   ~ 0
-SDO
 Wire Wire Line
-	13700 2850 14050 2850
-Wire Wire Line
-	13700 2950 14050 2950
+	3600 2800 4000 2800
+Text Label 4000 2800 2    50   ~ 0
+GPIO0
+Text Label 10900 3200 2    50   ~ 0
+RX_ESP32
 Wire Wire Line
-	14050 3050 13700 3050
+	10500 3200 10900 3200
 Wire Wire Line
-	13650 2300 14050 2300
-Text Label 13650 2300 0    49   ~ 0
-IO26
-Text Label 13650 2700 0    49   ~ 0
-IO33
-Text Label 13650 2600 0    49   ~ 0
-IO32
+	10200 4850 10650 4850
+Text Label 10650 4850 2    50   ~ 0
+GPIO0
+Text Label 1850 9200 2    50   ~ 0
+M2-
 Wire Wire Line
-	14050 2600 13650 2600
+	1400 9200 1850 9200
 $Comp
-L Connector_Generic:Conn_01x05 J7
-U 1 1 5FA2B066
-P 14250 2500
-F 0 "J7" H 14330 2542 50  0000 L CNN
-F 1 "Conn_01x05" H 14330 2451 50  0000 L CNN
-F 2 "Connector_PinHeader_2.54mm:PinHeader_1x05_P2.54mm_Vertical" H 14250 2500 50  0001 C CNN
-F 3 "~" H 14250 2500 50  0001 C CNN
-	1    14250 2500
+L power:GND #PWR022
+U 1 1 5F349ABA
+P 3000 5650
+F 0 "#PWR022" H 3000 5400 50  0001 C CNN
+F 1 "GND" H 3005 5477 50  0000 C CNN
+F 2 "" H 3000 5650 50  0001 C CNN
+F 3 "" H 3000 5650 50  0001 C CNN
+	1    3000 5650
 	1    0    0    -1
 $EndComp
-Text Label 13650 2500 0    49   ~ 0
-IO25
-Text Label 13650 2400 0    49   ~ 0
-IO27
-Wire Wire Line
-	14050 2500 13650 2500
-Wire Wire Line
-	14050 2400 13650 2400
-Wire Wire Line
-	14050 2700 13650 2700
+Wire Notes Line
+	15850 650  15850 3600
+Wire Notes Line
+	12100 3600 12100 650
+Wire Notes Line
+	15850 3600 12100 3600
 $EndSCHEMATC

Commit message: Routed completed Ready to order I hope
Parts:
- U3, U5, U8, U9: symbol Drone_Lib:SI2302-TP -> Drone_PCB-rescue:SI2302-TP-Drone_Lib
Changed lines of the file:
@@
 EESchema Schematic File Version 4
-LIBS:Drone_PCB-cache
 EELAYER 30 0
 EELAYER END
@@
 	3600 5000 3900 5000
 $Comp
-L Drone_Lib:SI2302-TP U8
+L Drone_PCB-rescue:SI2302-TP-Drone_Lib U8
 U 1 1 5F6DDDB5
 P 9000 8350
@@
 	8750 8200 9300 8200
 $Comp
-L Drone_Lib:SI2302-TP U9
+L Drone_PCB-rescue:SI2302-TP-Drone_Lib U9
 U 1 1 5F849D31
 P 10600 8400
@@
 	10350 8250 10900 8250
 $Comp
-L Drone_Lib:SI2302-TP U5
+L Drone_PCB-rescue:SI2302-TP-Drone_Lib U5
 U 1 1 5F8B4C53
 P 7450 8350
@@
 	7200 8200 7750 8200
 $Comp
-L Drone_Lib:SI2302-TP U3
+L Drone_PCB-rescue:SI2302-TP-Drone_Lib U3
 U 1 1 5F8C55B7
 P 5950 8300
