File: Battery Charger/Battery Charger.kicad_pcb (KiCad board)
At the start: 2 copper layers, 20 x 20 mm, 8 parts, among them J1 USB_B_Micro, J2 Conn_01x02, U1 MCP73831-2-OT

Commit message: Updated Latest
Parts:
- added FD1: Fiducial_0.75mm_Mask1.5mm, Fiducial:Fiducial_0.75mm_Mask1.5mm, F.Cu at (67.9, 96.2)
- added FD2: Fiducial_0.75mm_Mask1.5mm, Fiducial:Fiducial_0.75mm_Mask1.5mm, F.Cu at (82.0, 79.4)
Changed lines of the file:
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@@
-(kicad_pcb (version 20171130) (host pcbnew "(5.1.4)-1")
+(kicad_pcb (version 20171130) (host pcbnew "(5.1.5)-3")
   (general
     (thickness 1.6)
@@
     (tracks 66)
     (zones 0)
-    (modules 8)
+    (modules 10)
     (nets 10)
   )
@@
     (pad_to_mask_clearance 0.051)
     (solder_mask_min_width 0.25)
-    (aux_axis_origin 0 0)
-    (visible_elements FFFFFF7F)
+    (aux_axis_origin 81.407 79.248)
+    (grid_origin 65.151 97.917)
+    (visible_elements 7FFFFFFF)
     (pcbplotparams
       (layerselection 0x010fc_ffffffff)
@@
     (add_net V_BATT)
   )
+  (module Fiducial:Fiducial_0.75mm_Mask1.5mm (layer F.Cu)
+    (at 67.8815 96.2025)
+    (descr "Circular Fiducial, 0.75mm bare copper, 1.5mm soldermask opening (Level B)")
+    (tags fiducial)
+    (attr smd)
+    (fp_text reference FD1 (at 0 -2) (layer F.SilkS)
+      (effects (font (size 1 1) (thickness 0.15)))
+    )
+    (fp_text value Fiducial_0.75mm_Mask1.5mm (at 0 2) (layer F.Fab)
+      (effects (font (size 1 1) (thickness 0.15)))
+    )
+    (fp_circle (center 0 0) (end 0.75 0) (layer F.Fab) (width 0.1))
+    (fp_text user %R (at 0 0) (layer F.Fab)
+      (effects (font (size 0.3 0.3) (thickness 0.05)))
+    )
+    (fp_circle (center 0 0) (end 1 0) (layer F.CrtYd) (width 0.05))
+    (pad "" smd circle (at 0 0) (size 0.75 0.75) (layers F.Cu F.Mask)
+      (solder_mask_margin 0.375) (clearance 0.375))
+  )
+  (module Fiducial:Fiducial_0.75mm_Mask1.5mm (layer F.Cu)
+    (at 82.042 79.4385)
+    (descr "Circular Fiducial, 0.75mm bare copper, 1.5mm soldermask opening (Level B)")
+    (tags fiducial)
+    (attr smd)
+    (fp_text reference FD2 (at 2.032 0 90) (layer F.SilkS)
+      (effects (font (size 1 1) (thickness 0.15)))
+    )
+    (fp_text value Fiducial_0.75mm_Mask1.5mm (at 0 2) (layer F.Fab)
+      (effects (font (size 1 1) (thickness 0.15)))
+    )
+    (fp_circle (center 0 0) (end 1 0) (layer F.CrtYd) (width 0.05))
+    (fp_text user %R (at 0 0) (layer F.Fab)
+      (effects (font (size 0.3 0.3) (thickness 0.05)))
+    )
+    (fp_circle (center 0 0) (end 0.75 0) (layer F.Fab) (width 0.1))
+    (pad "" smd circle (at 0 0) (size 0.75 0.75) (layers F.Cu F.Mask)
+      (solder_mask_margin 0.375) (clearance 0.375))
+  )
   (module Connector_USB:USB_Micro-B_Molex-105017-0001 (layer F.Cu)
     (at 75.438 80.645 180)
@@
       (rotate (xyz 0 0 0))
     )
-    (model "C:/Users/kerip/Downloads/MOLEX_1050170001 (1)/1050170001.stp"
-      (offset (xyz 0 -1 1.2))
+    (model "D:/KiCad/Step Files/USB/1050170001.stp"
+      (offset (xyz 0 -1 1.5))
       (scale (xyz 1 1 1))
       (rotate (xyz -90 0 0))
@@
     (effects (font (size 1 1) (thickness 0.15)))
   )
-  (gr_text USB (at 82.423 79.375) (layer F.SilkS)
+  (gr_text USB (at 67.564 78.9305) (layer F.SilkS)
     (effects (font (size 1.5 1.5) (thickness 0.15)))
   )
@@
   (segment (start 71.882 86.995) (end 72.136 86.741) (width 0.25) (layer F.Cu) (net 1))
   (segment (start 72.136 86.741) (end 73.431 86.741) (width 0.25) (layer F.Cu) (net 1))
-  (segment (start 78.5835 87.691) (end 78.613 87.7205) (width 0.25) (layer F.Cu) (net 2))
-  (segment (start 76.411 87.691) (end 78.5835 87.691) (width 0.25) (layer F.Cu) (net 2))
-  (segment (start 81.788 85.9425) (end 81.788 88.0475) (width 0.25) (layer F.Cu) (net 4))
   (segment (start 72.538 79.4075) (end 78.938 79.4075) (width 0.25) (layer F.Cu) (net 1))
   (segment (start 71.938 81.1075) (end 71.938 79.4075) (width 0.25) (layer F.Cu) (net 1))
@@
   (segment (start 75.936 93.019) (end 76.526 93.019) (width 0.25) (layer F.Cu) (net 1))
   (segment (start 76.526 93.019) (end 76.9255 92.6195) (width 0.25) (layer F.Cu) (net 1))
+  (segment (start 78.5835 87.691) (end 78.613 87.7205) (width 0.25) (layer F.Cu) (net 2))
+  (segment (start 76.411 87.691) (end 78.5835 87.691) (width 0.25) (layer F.Cu) (net 2))
   (segment (start 78.613 90.551) (end 78.613 87.7205) (width 0.25) (layer F.Cu) (net 2))
   (segment (start 81.788 91.0225) (end 79.0845 91.0225) (width 0.25) (layer F.Cu) (net 2))
@@
   (segment (start 74.686 93.019) (end 74.223 93.019) (width 0.25) (layer F.Cu) (net 3))
   (segment (start 74.223 93.019) (end 73.9505 92.7465) (width 0.25) (layer F.Cu) (net 3))
+  (segment (start 81.788 85.9425) (end 81.788 88.0475) (width 0.25) (layer F.Cu) (net 4))
   (segment (start 76.206 85.791) (end 75.0335 84.6185) (width 0.25) (layer F.Cu) (net 8))
   (segment (start 75.0335 84.6185) (end 71.882 84.6185) (width 0.25) (layer F.Cu) (net 8))

Commit message: Updated Macro Keyboard
Parts:
- removed FD1, FD2: Fiducial_0.75mm_Mask1.5mm, Fiducial:Fiducial_0.75mm_Mask1.5mm
- added REF**: Fiducial_0.5mm_Mask1.5mm, Fiducial:Fiducial_0.5mm_Mask1.5mm, F.Cu at (67.8, 95.8)
- added REF**: Fiducial_0.5mm_Mask1.5mm, Fiducial:Fiducial_0.5mm_Mask1.5mm, F.Cu at (82.0, 79.6)
Routing:
- net /STAT: track 10.8 -> 25.6 mm
- net VBUS: track 27.6 -> 15.4 mm
- net GND: track 38.3 -> 47.2 mm, vias 2 -> 0
- net V_BATT: track 6.01 -> 6.95 mm
- added copper zone on F.Cu, net V_BATT
- removed copper zone on F.Cu, net VBUS
Other:
- board size 20 x 20 mm -> 19.9 x 20.2 mm
- net class VBat_Width added: clearance 0.2, trace_width 0.5, via_dia 0.8, via_drill 0.4
- net class Vbus_Width added: clearance 0.2, trace_width 0.5, via_dia 0.8, via_drill 0.4
